Commit message: gazebo worls and realsense positioning

File: xarm_description/urdf/camera/realsense_d435i.urdf.xacro (robot description, xacro)
@@ -5,4 +5,6 @@
     <xacro:property name="M_PI" value="3.1415926535897931" />
     <link name="${prefix}link_eef">
+    </link>
+    <link name="${prefix}link_eef_static">
       <xacro:common_link_visual
         mesh_filename="camera/realsense/visual/d435_with_cam_stand"
@@ -26,5 +28,5 @@
       <link name="${prefix}camera_right_ir_optical_frame"></link>
       <joint name="${prefix}camera_link_joint" type="fixed">
-        <parent link="${prefix}link_eef" />
+        <parent link="${prefix}link_eef_static" />
         <child link="${prefix}camera_link" />
         <origin xyz="0.06746 -0.0175 0.0237" rpy="${M_PI} ${-M_PI/2} 0" />

File: xarm_description/urdf/xarm_device_macro.xacro (robot description, xacro)
@@ -47,4 +47,6 @@
     <xacro:include filename="$(find xarm_description)/urdf/_private_macro.xacro" />
     <xacro:device_macro_begin />
+    <!-- define property -->
+    <xacro:property name="M_PI" value="3.1415926535897931" />
     <!-- Load Common Material -->
     <xacro:include filename="$(find xarm_description)/urdf/common/common.material.xacro" />
@@ -217,4 +219,9 @@
       <parent link="${prefix}link${dof}" />
       <child link="${prefix}link_eef" />
+    </joint>
+    <joint name="${prefix}camera_static" type="fixed">
+      <parent link="${prefix}link_base" />
+      <child link="${prefix}link_eef_static" />
+      <origin xyz="-0.3 0.0 2.0" rpy="0 ${M_PI} 0" />
     </joint>
     <xacro:if value="${add_gripper}">

Commit message: added sattic camera

File: xarm_description/urdf/camera/realsense_d435i.urdf.xacro (robot description, xacro)
@@ -1,10 +1,8 @@
 <?xml version="1.0"?>
-<robot xmlns:xacro="http://ros.org/wiki/xacro">
+<robot name="camera_gripper" xmlns:xacro="http://ros.org/wiki/xacro">
   <xacro:macro name="d435i_urdf" params="prefix:='' add_d435i_links:=false">
     <!-- define property -->
     <xacro:property name="M_PI" value="3.1415926535897931" />
     <link name="${prefix}link_eef">
-    </link>
-    <link name="${prefix}link_eef_static">
       <xacro:common_link_visual
         mesh_filename="camera/realsense/visual/d435_with_cam_stand"
@@ -28,5 +26,5 @@
       <link name="${prefix}camera_right_ir_optical_frame"></link>
       <joint name="${prefix}camera_link_joint" type="fixed">
-        <parent link="${prefix}link_eef_static" />
+        <parent link="${prefix}link_eef" />
         <child link="${prefix}camera_link" />
         <origin xyz="0.06746 -0.0175 0.0237" rpy="${M_PI} ${-M_PI/2} 0" />

File: xarm_description/urdf/camera_static/realsense_static.gazebo.xacro (robot description, xacro)
@@ -1,8 +1,8 @@
 <?xml version="1.0"?>
-<robot name="camera_dynamic" xmlns:xacro="http://ros.org/wiki/xacro">
-  <xacro:macro name="realsense_gazebo" params="prefix:='' ">
-    <gazebo reference="${prefix}camera_depth_frame">
+<robot name="camera_static" xmlns:xacro="http://ros.org/wiki/xacro">
+  <xacro:macro name="realsense_static_gazebo" params="prefix:='' ">
+    <gazebo reference="${prefix}camera_static_depth_frame">
       <sensor name="cameradepth" type="depth">
-        <camera name="camera">
+        <camera name="camera_static">
           <horizontal_fov>1.57</horizontal_fov>
           <image>
@@ -25,7 +25,7 @@
       </sensor>
     </gazebo>
-    <gazebo reference="${prefix}camera_color_frame">
+    <gazebo reference="${prefix}camera_static_color_frame">
       <sensor name="cameracolor" type="camera">
-        <camera name="camera">
+        <camera name="camera_static">
           <horizontal_fov>1.57</horizontal_fov>
           <image>
@@ -49,7 +49,7 @@
       </sensor>
     </gazebo>
-    <gazebo reference="${prefix}camera_left_ir_frame">
+    <gazebo reference="${prefix}camera_static_left_ir_frame">
       <sensor name="cameraired1" type="camera">
-        <camera name="camera">
+        <camera name="camera_static">
           <horizontal_fov>1.57</horizontal_fov>
           <image>
@@ -73,7 +73,7 @@
       </sensor>
     </gazebo>
-    <gazebo reference="${prefix}camera_right_ir_frame">
+    <gazebo reference="${prefix}camera_static_right_ir_frame">
       <sensor name="cameraired2" type="camera">
-        <camera name="camera">
+        <camera name="camera_static">
           <horizontal_fov>1.57</horizontal_fov>
           <image>
@@ -103,20 +103,20 @@
         <colorUpdateRate>30.0</colorUpdateRate>
         <infraredUpdateRate>30.0</infraredUpdateRate>
-        <depthTopicName>aligned_depth_to_color/image_raw</depthTopicName>
-        <depthCameraInfoTopicName>depth/camera_info</depthCameraInfoTopicName>
-        <colorTopicName>color/image_raw</colorTopicName>
-        <colorCameraInfoTopicName>color/camera_info</colorCameraInfoTopicName>
-        <infrared1TopicName>infra1/image_raw</infrared1TopicName>
-        <infrared1CameraInfoTopicName>infra1/camera_info</infrared1CameraInfoTopicName>
-        <infrared2TopicName>infra2/image_raw</infrared2TopicName>
-        <infrared2CameraInfoTopicName>infra2/camera_info</infrared2CameraInfoTopicName>
-        <colorOpticalframeName>camera_color_optical_frame</colorOpticalframeName>
-        <depthOpticalframeName>camera_depth_optical_frame</depthOpticalframeName>
-        <infrared1OpticalframeName>camera_left_ir_optical_frame</infrared1OpticalframeName>
-        <infrared2OpticalframeName>camera_right_ir_optical_frame</infrared2OpticalframeName>
+        <depthTopicName>aligned_depth_to_color_static/image_raw_static</depthTopicName>
+        <depthCameraInfoTopicName>depth_static/camera_info_static</depthCameraInfoTopicName>
+        <colorTopicName>color_static/image_raw_static</colorTopicName>
+        <colorCameraInfoTopicName>color_static/camera_info_static</colorCameraInfoTopicName>
+        <infrared1TopicName>infra1_static/image_raw_static</infrared1TopicName>
+        <infrared1CameraInfoTopicName>infra1_static/camera_info_static</infrared1CameraInfoTopicName>
+        <infrared2TopicName>infra2_static/image_raw_static</infrared2TopicName>
+        <infrared2CameraInfoTopicName>infra2_static/camera_info_static</infrared2CameraInfoTopicName>
+        <colorOpticalframeName>camera_color_optical_frame_static</colorOpticalframeName>
+        <depthOpticalframeName>camera_depth_optical_frame_static</depthOpticalframeName>
+        <infrared1OpticalframeName>camera_left_ir_optical_frame_static</infrared1OpticalframeName>
+        <infrared2OpticalframeName>camera_right_ir_optical_frame_static</infrared2OpticalframeName>
         <rangeMinDepth>0.3</rangeMinDepth>
         <rangeMaxDepth>3.0</rangeMaxDepth>
         <pointCloud>true</pointCloud>
-        <pointCloudTopicName>depth/color/points</pointCloudTopicName>
+        <pointCloudTopicName>depth_static/color/points</pointCloudTopicName>
         <pointCloudCutoff>0.3</pointCloudCutoff>
       </plugin>

File: xarm_description/urdf/xarm_device_macro.xacro (robot description, xacro)
@@ -220,8 +220,20 @@
       <child link="${prefix}link_eef" />
     </joint>
-    <joint name="${prefix}camera_static" type="fixed">
+    <xacro:if value="${add_realsense_d435i}">
+      <!-- (xarm) Load RealSense D435i URDF -->
+      <xacro:include filename="$(find xarm_description)/urdf/camera_static/realsense_d435i_static.urdf.xacro" />
+      <xacro:d435i_static_urdf prefix="${prefix}" add_d435i_links="${add_d435i_links}" />
+      <xacro:if value="${add_d435i_links}">
+        <xacro:include filename="$(find xarm_description)/urdf/camera_static/realsense_static.gazebo.xacro" />
+        <xacro:realsense_static_gazebo prefix="${prefix}" />
+      </xacro:if>
+    </xacro:if>
+    <xacro:unless value="${add_realsense_d435i}">
+      <link name="${prefix}link_eef_static"/>
+    </xacro:unless>
+    <joint name="${prefix}joint_eef_static" type="fixed">
+      <origin xyz="-0.3 0.0 2.0" rpy="0 ${M_PI} 0" />
       <parent link="${prefix}link_base" />
       <child link="${prefix}link_eef_static" />
-      <origin xyz="-0.3 0.0 2.0" rpy="0 ${M_PI} 0" />
     </joint>
     <xacro:if value="${add_gripper}">
